File: hardware/rapidshark-main-breakout-top-mk-1.7-fab.brd (EAGLE design)
At the start: 44 x 18 mm, 13 parts, among them U1 ADAFRUIT_METRO_MININOSILK-AMB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

Commit message: renaming nets so i can copypasta into the sketch
Connections:
- net ACCEL renamed SW_ACCEL
- net CLIP renamed SW_CLIP
- net DART renamed DART_DETECT
- net FIRE renamed SW_FIRE
- net PUSH renamed SW_PUSH
- net X renamed BUTT_X
- net Y renamed BUTT_Y
- net Z renamed BUTT_Z
Changed lines of the file:
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@@
 <setting verticaltext="up"/>
 </settings>
-<grid distance="0.25" unitdist="mm" unit="mm" style="lines" multiple="2" display="yes" altdistance="1" altunitdist="mil" altunit="mil"/>
+<grid distance="0.5" unitdist="mm" unit="mm" style="lines" multiple="2" display="yes" altdistance="1" altunitdist="mil" altunit="mil"/>
 <layers>
 <layer number="1" name="Top" color="4" fill="1" visible="yes" active="yes"/>
@@
 <wire x1="10.316" y1="1.634" x2="10.316" y2="4.8" width="0.5" layer="16"/>
 </signal>
-<signal name="DART">
+<signal name="DART_DETECT">
 <contactref element="CLIP" pad="3"/>
 <contactref element="U1" pad="3"/>
@@
 <wire x1="32" y1="14.5" x2="32" y2="9.5" width="0.3" layer="16"/>
 </signal>
-<signal name="CLIP">
+<signal name="SW_CLIP">
 <contactref element="CLIP" pad="4"/>
 <contactref element="U1" pad="5"/>
@@
 <wire x1="28.5" y1="6" x2="29" y2="6" width="0.3" layer="16"/>
 </signal>
-<signal name="PUSH">
+<signal name="SW_PUSH">
 <contactref element="TRIG" pad="2"/>
 <contactref element="U1" pad="4"/>
@@
 <wire x1="24.27" y1="10" x2="30.89" y2="16.62" width="0.3" layer="1"/>
 </signal>
-<signal name="FIRE">
+<signal name="SW_FIRE">
 <contactref element="TRIG" pad="3"/>
 <contactref element="U1" pad="6"/>
@@
 <wire x1="22.5" y1="8" x2="23" y2="8" width="0.3" layer="1"/>
 </signal>
-<signal name="ACCEL">
+<signal name="SW_ACCEL">
 <contactref element="TRIG" pad="4"/>
 <contactref element="U1" pad="7"/>
@@
 <wire x1="20.73" y1="2.77" x2="20.73" y2="1.38" width="0.5" layer="1"/>
 </signal>
-<signal name="X">
+<signal name="BUTT_X">
 <contactref element="U1" pad="25"/>
 <contactref element="BUTT" pad="4"/>
@@
 <wire x1="30.89" y1="1.89" x2="35" y2="6" width="0.3" layer="16"/>
 </signal>
-<signal name="Y">
+<signal name="BUTT_Y">
 <contactref element="U1" pad="24"/>
 <contactref element="BUTT" pad="3"/>
@@
 <wire x1="28.38" y1="1.38" x2="35" y2="8" width="0.3" layer="16"/>
 </signal>
-<signal name="Z">
+<signal name="BUTT_Z">
 <contactref element="U1" pad="23"/>
 <contactref element="BUTT" pad="2"/>
