File: hardware/rapidshark-main-breakout-top-mk-1.7-fab.sch (EAGLE design)
At the start: 11 parts, among them U1 ADAFRUIT_METRO_MININOSILK-AMB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

Commit message: renaming nets so i can copypasta into the sketch
Connections:
- net ACCEL renamed SW_ACCEL
- net CLIP renamed SW_CLIP
- net DART renamed DART_DETECT
- net FIRE renamed SW_FIRE
- net PUSH renamed SW_PUSH
- net X renamed BUTT_X
- net Y renamed BUTT_Y
- net Z renamed BUTT_Z
Changed lines of the file:
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@@
 </segment>
 </net>
-<net name="DART" class="0">
+<net name="DART_DETECT" class="0">
 <segment>
 <pinref part="CLIP" gate="G$1" pin="3"/>
@@
 </segment>
 </net>
-<net name="CLIP" class="0">
+<net name="SW_CLIP" class="0">
 <segment>
 <pinref part="CLIP" gate="G$1" pin="4"/>
@@
 </segment>
 </net>
-<net name="PUSH" class="0">
+<net name="SW_PUSH" class="0">
 <segment>
 <pinref part="TRIG" gate="G$1" pin="2"/>
@@
 </segment>
 </net>
-<net name="FIRE" class="0">
+<net name="SW_FIRE" class="0">
 <segment>
 <pinref part="TRIG" gate="G$1" pin="3"/>
@@
 </segment>
 </net>
-<net name="ACCEL" class="0">
+<net name="SW_ACCEL" class="0">
 <segment>
 <pinref part="TRIG" gate="G$1" pin="4"/>
@@
 </segment>
 </net>
-<net name="X" class="0">
+<net name="BUTT_X" class="0">
 <segment>
 <wire x1="73.66" y1="144.78" x2="71.12" y2="144.78" width="0.1524" layer="91"/>
@@
 </segment>
 </net>
-<net name="Y" class="0">
+<net name="BUTT_Y" class="0">
 <segment>
 <wire x1="73.66" y1="142.24" x2="71.12" y2="142.24" width="0.1524" layer="91"/>
@@
 </segment>
 </net>
-<net name="Z" class="0">
+<net name="BUTT_Z" class="0">
 <segment>
 <wire x1="73.66" y1="139.7" x2="71.12" y2="139.7" width="0.1524" layer="91"/>
