File: hardware/rapidshark-main-breakout-top-mk-1.A.brd (EAGLE design)
At the start: 44 x 18 mm, 14 parts, among them U1 ADAFRUIT_METRO_MINIBIGHOLES

Commit message: finishing resistor add layout
Connections:
- net 3.3V: now also DSPLY.1; no longer DSPLY.3
- net DISP_RST: now also DSPLY.6; no longer DSPLY.4
- net GND: now also DSPLY.3; no longer DSPLY.1
- net SCL: now also DSPLY.5; no longer DSPLY.6
- net SDA: now also DSPLY.4; no longer DSPLY.5
Routing:
- net SCL: track 4.46 -> 9.49 mm
- net 5V: track 66.4 -> 70.0 mm
- net 3.3V: track 36.5 -> 40.0 mm
- net DISP_RST: track 12.0 -> 8.86 mm, vias 1 -> 0
- net N$1: track 24.1 -> 24.6 mm
