File: hardware/rapidshark-main-breakout-top-mk-1.A.sch (EAGLE design)
At the start: 12 parts, among them U1 ADAFRUIT_METRO_MINIBIGHOLES

Commit message: finishing resistor add layout
Parts:
- FRAME1: VERSION v1.B -> v1.A
Connections:
- net 3.3V: now also DSPLY.1; no longer DSPLY.3
- net DISP_RST: now also DSPLY.6; no longer DSPLY.4
- net GND: now also DSPLY.3; no longer DSPLY.1
- net SCL: now also DSPLY.5; no longer DSPLY.6
- net SDA: now also DSPLY.4; no longer DSPLY.5
Other:
- moved on the sheet: DSPLY
