File: hardware/rapidshark-lipo-sensor-mk-1.1.brd (EAGLE design)
At the start: 35.6 x 20.3 mm, 13 parts, among them IC1 Tiny84, Q1 2N7000, Q2 2N7000, Q3 2N7000

Commit message: lipo voltage testing boards
Parts:
- removed C0: 100n, A_butts:C025-024X044
- removed IC1: Tiny84, A_butts:DIL14
- removed Q1, Q2, Q3: 2N7000, a_parts:TO-92
- removed R0, R2, R3, R4: 10k, A_butts:RESISTOR-AXIAL-PTH-5.08MM
- added C1: 100n, A_butts:C025-024X044
- added U1: TINY85, A_butts:DIP08
- R1: device A_butts:RESISTOR-AXIAL-PTH-5.08MM -> A_butts:RESISTOR-AXIAL-PTH-7.62MM
- moved AVRISP 47.0 mm to (6.99, -23.2)
- moved BATT 46.4 mm to (1.59, -40.0), turned to 0 degrees
- moved R1 33.3 mm to (11.4, -27.0), turned to 0 degrees
Connections:
- removed net BATT-: BATT.1, R1.P$2
- removed net EN1: IC1.2, Q1.2
- removed net EN2: IC1.3, Q2.2
- removed net EN3: IC1.5, Q3.2
- removed net N$3: Q3.3, R4.P$1
- removed net VDIV3: IC1.10, Q2.3, Q3.1, R3.P$1
- net CELL1+: no longer R2.P$2
- net CELL2+: no longer R3.P$2
- net CELL3+: no longer R4.P$2
- net GND: now also BATT.1, C1.2, U1.4; no longer C0.2, IC1.14
- net MISO: now also U1.6; no longer IC1.8
- net MOSI/SDA: now also U1.5; no longer IC1.7
- net RESET: now also R1.P$1, U1.1; no longer IC1.4, R0.P$1
- net SCK/SCL: now also U1.7; no longer IC1.9
- net VCC: now also C1.1, R1.P$2, U1.8; no longer C0.1, IC1.1, R0.P$2
- net VDIV1: now also U1.2; no longer IC1.12, Q1.1, R1.P$1
- net VDIV2: now also U1.3; no longer IC1.11, Q1.3, Q2.1, R2.P$1
Other:
- board size 35.6 x 20.3 mm -> 27.9 x 16.5 mm
- board text added: "2S Lipo Voltmeter"
- board text added: "by schizobovine"
