File: hardware/rapidshark-lipo-sensor-mk-1.1.sch (EAGLE design)
At the start: 13 parts, among them IC1 Tiny84, Q1 2N7000, Q2 2N7000, Q3 2N7000

Commit message: lipo voltage testing boards
Parts:
- removed C0: 100n, A_butts:CAPACITOR-CERAMIC025-024X044
- removed IC1: Tiny84, A_butts:ATTINY84ATTINY84-20PU
- removed Q1, Q2, Q3: 2N7000, a_parts:MOSFET-NCHANNEL2N7000
- removed R0, R2, R3, R4: 10k, A_butts:RESISTORPTH-AXIAL-5.08MM
- added C1: 100n, A_butts:CAPACITOR-CERAMIC025-024X044
- added U1: TINY85, A_butts:ATTINY45TINY85-20-DIP
- FRAME1: VERSION v2.0 -> v1.0
- R1: device A_butts:RESISTORPTH-AXIAL-5.08MM -> A_butts:RESISTORPTH-AXIAL-7.62MM
Connections:
- removed net BATT-: BATT.1, R1.2
- removed net EN1: IC1.(PCINT8/XTAL1/CLKI)PB0, Q1.G
- removed net EN2: IC1.(PCINT9/XTAL2)PB1, Q2.G
- removed net EN3: IC1.(PCINT10/INT0/OC0A/CKOUT)PB2, Q3.G
- removed net N$3: Q3.D, R4.1
- removed net VDIV3: IC1.(PCINT3/T0/ADC3)PA3, Q2.D, Q3.S, R3.1
- net CELL1+: no longer R2.2
- net CELL2+: no longer R3.2
- net CELL3+: no longer R4.2
- net GND: now also BATT.1, C1.2, U1.GND; no longer C0.2, IC1.GND
- net MISO: now also U1.PB1(MISO); no longer IC1.(PCINT5/OC1B/MISO/DO/ADC5)PA5
- net MOSI/SDA: now also U1.PB0(MOSI); no longer IC1.(PCINT6/OC1A/SDA/MOSI/ADC6)PA6
- net RESET: now also R1.1, U1.RESET; no longer IC1.(PCINT11/~RESET/DW)PB3, R0.1
- net SCK/SCL: now also U1.PB2(SCK/ADC1); no longer IC1.(PCINT4/T1/SCL/USCK/ADC4)PA4
- net VCC: now also C1.1, R1.2, U1.VCC; no longer C0.1, IC1.VCC, R0.2
- net VDIV1: now also U1.PB3(ADC3); no longer IC1.(PCINT1/AIN0/ADC1)PA1, Q1.S, R1.1
- net VDIV2: now also U1.PB4(ADC2); no longer IC1.(PCINT2/AIN1/ADC2)PA2, Q1.D, Q2.S, R2.1
Other:
- moved on the sheet: AVRISP, BATT, R1
