File: hardware/rapidshark-half-assed-half-h-bridge-mk-3.0.sch (EAGLE design)
At the start: 28 parts, among them Q2 IRF540N

Commit message: WIP A3946 half bridge driver
Parts:
- removed R6: 27R, a_parts:RESISTORR0603-TIGHTER
- removed R7, R8: 330R, a_parts:RESISTORR0603-TIGHTER
- removed SJ1: JUMPER-PAD-2-NO, a_parts:JUMPER-PAD-2-NO
- added C6, C7: 470uF, a_parts:CAPACITOR-POLARIZEDE5-10.5
- added IC1: A3946LP, a_parts:A3946LP
- added JP1: (no value), a_parts:JUMPER-PAD-3-NOFULL_BOX_SILK
- added Q1: IRLR3410, a_parts:MOSFET-NCHANNELFDD8780
- added R30, R70: 330R, a_parts:RESISTORR0603-TIGHTER
- C1: value 1uF -> 0.47uF
- C2: value 470uF -> 10uF; device a_parts:CAPACITOR-POLARIZEDE5-10.5 -> a_parts:CAPACITOR-CERAMICC0805-TIGHTER
- C3: value 470uF -> 0.1uF; device a_parts:CAPACITOR-POLARIZEDE5-10.5 -> a_parts:CAPACITOR-CERAMICC0603-TIGHTER
- C4: value 0.1uF -> 10uF; device a_parts:CAPACITOR-CERAMICC0603-TIGHTER -> a_parts:CAPACITOR-CERAMICC0805-TIGHTER
- C5: value 0.1uF -> 1uF
- Q2: value IRF540N -> IRLR3410
- R1: value 10k -> 10K
- R2: value 27R -> 15.8K
- R3, R4: value 330R -> 33R
- R5: value 10k -> 470K
Connections:
- removed net HS: HS.1, R3.1, R4.1
- removed net LS: LS.1, R7.1, R8.1
- new net !FAULT: IC1.!FAULT, R1.1
- new net IN1: IC1.IN1
- new net IN2: IC1.IN2
- new net N$11: IC1.GL, R4.1
- new net N$12: IC1.GH, R3.1
- new net RST: IC1.RESET
- new net VREF: C3.1, IC1.VREF, R1.2
- new net VREG: C4.1, IC1.VREG
- net A: now also C5.1, IC1.S, Q1.S, R5.1; no longer C1.1
- net GND: now also C3.2, C4.2, IC1.LGND, JP1.3, R2.1; no longer SJ1.1
- net N$1: now also R4.2; no longer R5.2, R6.2
- net N$2: now also C1.1, IC1.CP1; no longer R2.1
- net N$3: now also R70.2; no longer R7.2
- net N$4: now also R30.2; no longer R3.2
- net N$5: now also Q1.G, R3.2, R5.2; no longer R1.1, R2.2
- net N$6: now also C1.2, IC1.CP2; no longer R4.2
- net N$7: now also IC1.DT, R2.2; no longer R8.2
- net N$8: now also IC1.PAD, JP1.2; no longer R6.1
- net PGND: now also C2.2, C6.-, C7.-, IC1.PGND, JP1.1; no longer C1.2, C2.-, C3.-, C4.2, R5.1, SJ1.2
- net VBAT: now also C2.1, C6.+, C7.+, IC1.VBB, Q1.D; no longer C2.+, C3.+, C4.1, C5.1, R1.2
Other:
- moved on the sheet: +, -, A, B, C1, C4, C5, D1, D2, HI, LO, Q2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
