File: hardware/rapidshark-half-assed-half-h-bridge-mk-1.1.sch (EAGLE design)
At the start: 26 parts, among them Q1 SPD15P10PL, Q2 IRLR3410, Q3 MMBT2222A, Q4 MMBT4403, U1 ARDUINO_PRO_MINIMINE

Commit message: more twiddling around with cheap h-bridge ideas
Parts:
- added A2: M01PTH, a_parts:M01PTH
- +, -, A, B: value M01PTH-1.5MM -> M01PTH-1.4MM; device a_parts:M01PTH-1.5MM -> a_parts:M01PTH-1.4MM
- renumbered D5/HS to D11/LS, D6/LS to D10/HS
Connections:
- removed net V_BATT: +.1, D1.C, Q1.S, R1.2
- net GND: no longer U1.GND@2
- net HS: now also D10/HS.1; no longer D11/LS.1, U1.*5
- net LS: now also D11/LS.1; no longer D10/HS.1, U1.*6
- net VBAT: now also +.1, D1.C, Q1.S, R1.2; no longer U1.RAW
Other:
- moved on the sheet: D3, R3, U1
