File: hardware/rapidshark-half-assed-half-h-bridge-mk-1.4.brd (EAGLE design)
At the start: 20.3 x 35.6 mm, 29 parts, among them Q1 IRLR3410, Q2 IRLR3410, U1 Tiny85, U3 IR2304

Commit message: more bridge shenanigans
Parts:
- removed AVRISP: AVR_SPI_PRG_6SMD_TEST_POINTS, a_parts:2X3_SMD_TEST_POINTS
- removed C4: 10uF, a_parts:C0805-TIGHTER
- removed D3: BAT54JFILM, a_parts:SOD323-SCHOTTKY
- removed JP1: M03PTH-CENTERED, a_parts:1X03-CENTERED
- removed U2: (no value), a_parts:SOT23
- added 5V, GND, MISO, MOSI, RST, SCK: M01PTH-0.9MM, a_parts:1X01-0.9MM
- U$1: device a_parts:COW_SMALL_METAL_NOTEXT -> a_parts:COW_SMALL_NOTEXT
- U1: value Tiny85 -> TINY85
- moved U$2 32.0 mm to (5.08, 12.1)
- moved U$1 27.3 mm to (10.2, 28.6)
- moved U$3 27.1 mm to (14.5, 12.1), flipped to the bottom
- moved + 16.5 mm to (1.91, 33.7)
- moved A 16.5 mm to (18.4, 33.7)
- moved C3 14.5 mm to (16.5, 2.54), turned to 270 degrees
- moved C7 14.4 mm to (5.08, 15.2), turned to 0 degrees
- moved R2 12.2 mm to (18.5, 17.8), turned to 90 degrees
- moved U3 11.7 mm to (14.9, 14.0)
- moved U1 10.5 mm to (12.7, 5.08), turned to 180 degrees
- moved C2 10.2 mm to (15.2, 33.7), turned to 180 degrees
- moved C6 10.2 mm to (5.08, 33.7), turned to 0 degrees
- moved R1 8.93 mm to (11.2, 16.1), turned to 90 degrees
- moved C1 8.18 mm to (14.2, 19.1), turned to 0 degrees
- moved R3 5.39 mm to (16.5, 7.62), turned to 270 degrees
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Connections:
- removed net MISO: AVRISP.1, U1.6
- removed net N$6: C3.1, D3.C, U2.3
- new net MISO/CTRL: MISO.1, U1.6
- net 5V: now also 5V.1, C3.1; no longer AVRISP.2, C4.1, U2.2
- net GND: now also GND.1; no longer AVRISP.6, C4.2, U2.1
- net MOSI: now also MOSI.1; no longer AVRISP.4
- net RESET: now also RST.1; no longer AVRISP.5
- net SCK: now also SCK.1; no longer AVRISP.3
- net VBAT: no longer D3.A
Routing:
- net VBAT: track 0.00 -> 18.4 mm, vias 0 -> 33
- net RESET: track 0.00 -> 18.3 mm, vias 0 -> 1
- net 5V: track 0.00 -> 13.8 mm, vias 0 -> 1
- net N$1: track 0.00 -> 12.6 mm
- net MISO/CTRL: track 0.00 -> 12.4 mm, vias 0 -> 1
- net N$5: track 0.00 -> 12.2 mm, vias 0 -> 2
- net MOSI: track 0.00 -> 11.0 mm
- net SCK: track 0.00 -> 7.88 mm
- net N$2: track 0.00 -> 6.26 mm
- net N$3: track 0.00 -> 5.21 mm
- net GND: track 0.00 -> 4.85 mm
- net A: track 0.00 -> 3.58 mm, vias 0 -> 34
- net LS: track 0.00 -> 3.47 mm
- net HS: track 0.00 -> 3.47 mm
- net N$4: track 0.00 -> 1.96 mm
- added copper zone on layer 1, net A
- added copper zone on layer 16, net A
- added copper zone on layer 1, net VBAT
- added copper zone on layer 16, net VBAT
Other:
- outline, holes or cut-outs redrawn
