File: hardware/rapidshark-half-assed-half-h-bridge-mk-1.4.sch (EAGLE design)
At the start: 26 parts, among them Q1 IRLR3410, Q2 IRLR3410, U1 Tiny85, U3 IR2304

Commit message: more bridge shenanigans
Parts:
- removed AVRISP: AVR_SPI_PRG_6SMD_TEST_POINTS, a_parts:AVR_SPI_PRG_6SMD_TEST_POINTS
- removed C4: 10uF, a_parts:CAPACITOR-CERAMICC0805-TIGHTER
- removed D3: BAT54JFILM, a_parts:DIODE-SCHOTTKYSOD323
- removed JP1: M03PTH-CENTERED, a_parts:M03PTH-CENTERED
- removed U2: (no value), a_parts:VREG_1117SOT-23
- added 5V, GND, MISO, MOSI, RST, SCK: M01PTH-0.9MM, a_parts:M01PTH-0.9MM
- FRAME1: VERSION v1.3 -> v1.4
- U1: value Tiny85 -> TINY85
Connections:
- removed net MISO: AVRISP.MISO, U1.PB1(MISO)
- removed net N$6: C3.1, D3.C, U2.VIN
- new net MISO/CTRL: MISO.1, U1.PB1(MISO)
- net 5V: now also 5V.1, C3.1; no longer AVRISP.VCC, C4.1, U2.VOUT
- net GND: now also GND.1; no longer AVRISP.GND, C4.2, U2.GND
- net MOSI: now also MOSI.1; no longer AVRISP.MOSI
- net RESET: now also RST.1; no longer AVRISP.RST
- net SCK: now also SCK.1; no longer AVRISP.SCK
- net VBAT: no longer D3.A
Other:
- moved on the sheet: +, -, C3, C6, C7, C8
