File: hardware/rapidshark-main-breakout-top-mk-1.C.sch (EAGLE design)
At the start: 12 parts, among them U1 ADAFRUIT_METRO_MINIBIGHOLES

Commit message: asdlkfjaklsdfjsdlk
Parts:
- added JP1: M03JST-PTH-VERT, a_parts:M03JST-PTH-VERT
- ACCEL, PUSHER: device A_butts:M06JST-PH-PTH-VERT -> a_parts:M06JST-PH-PTH-VERT
- BUTT, CLIP, DISP, TRIG: device A_butts:M04JST-PTH-VERT -> a_parts:M04JST-PTH-VERT
- F1: device A_butts:PTCSMD -> a_parts:PTCSMD
- FRAME1: device A_butts:FRAME-LETTERNO_PACKAGE -> a_parts:FRAME-LETTERNO_PACKAGE
- R1, R2: device A_butts:RESISTORR0805 -> a_parts:RESISTORR0603-TIGHTER
- TVS: device A_butts:TVSSMA -> a_parts:TVSSMA
- U1: device A_butts:ADAFRUIT_METRO_MINIBIGHOLES -> a_parts:ADAFRUIT_METRO_MINIBIGHOLES
Connections:
- removed net ACCEL_A: ACCEL.1, U1.D8
- removed net ACCEL_B: ACCEL.3, U1.D10
- new net N$2: U1.D8
- new net N$3: U1.D10
- new net N$4: U1.D13
- net 5V: now also ACCEL.5, DISP.2; no longer ACCEL.4, DISP.1
- net GND: now also ACCEL.6, DISP.1; no longer ACCEL.5, DISP.2, U1.A3
Other:
- moved on the sheet: ACCEL, DISP

Commit message: new connector board for new motor driver and lipo sensor
Parts:
- removed BUTT: M04JST-PTH-VERT, a_parts:M04JST-PTH-VERT
- removed JP1: M03JST-PTH-VERT, a_parts:M03JST-PTH-VERT
- added FWD_IO: M04JST-PTH-VERT, a_parts:M04JST-PTH-VERT
- added RST: SPST-NO-TACTCK-PTS840-GK, a_parts:SPST-NO-TACTCK-PTS840-GK
- ACCEL: value M06JST-PH-PTH-VERT -> M03JST-PTH-VERT-CENTERED; device a_parts:M06JST-PH-PTH-VERT -> a_parts:M03JST-PTH-VERT-CENTERED
- TVS: value (none) -> 15V
Connections:
- removed net N$2: U1.D8
- removed net N$3: U1.D10
- removed net N$4: U1.D13
- removed net X: BUTT.4, U1.A2
- removed net Y: BUTT.3, U1.A1
- removed net Z: BUTT.2, U1.A0
- new net BMON_CLK: FWD_IO.4, U1.D13
- new net BMON_MISO: FWD_IO.3, U1.D12
- new net BMON_MOSI: FWD_IO.2, U1.D10
- new net BUTT: FWD_IO.1, U1.A0
- new net RESET: RST.1, U1.RST
- net 5V: now also ACCEL.1; no longer ACCEL.5
- net ACCEL_PWM: now also U1.D3; no longer U1.D9
- net DART: now also U1.D8; no longer U1.D2
- net GND: now also ACCEL.3, RST.2; no longer ACCEL.6, BUTT.1
- net PUSH: now also U1.D2; no longer U1.D3
- net PUSH_B: now also U1.D9; no longer U1.D12
Other:
- moved on the sheet: F1, TVS
