File: hardware/rapidshark-main-breakout-top-teensy-mk-1.1.sch (EAGLE design)
At the start: 16 parts, among them U1 TEENSY-3.1-OUTERPTH, U3 SN74LVC1T45SOT23-6

Commit message: new teensy lc mainboard with vreg
Parts:
- added C2: 2.2uF, a_parts:CAPACITOR-CERAMICC0603-TIGHTER
- added U2: MIC5235, a_parts:V_REG_MIC5235
- FRAME1: VERSION v1.E -> v1.F
- renumbered PSHR to PSH
Connections:
- net 5V: now also C2.1, U1.VIN, U2.OUT
- net GND: now also C2.2, U2.GND
- net VIN: now also U2.EN, U2.IN; no longer U1.VIN
Other:
- note added: "Reverse polarity protection from VNH5019's VOUT"
- note added: "VIN = 3S Lipo 11.1V nominal (9.0V min - 12.6V max/full)"
- note added: "VRAW = 3S Lipo 11.1V nominal (9.0V min - 12.6V max/full)"
- moved on the sheet: 3/17, BYPASS, C1, F1, PROG, R1, R2, TVS, U3
